File: MiniBench/MiniBench.kicad_pcb (KiCad board)
At the start: 2 copper layers, 30 x 18.5 mm, 27 parts, among them J1 10174819-00011LF, J3 Screw_Terminal_01x04, U1 AP2112K-1.8, U2 AMS1117-3.3

Commit message: Update README
Parts:
- removed H1, H2: M2, MountingHole:MountingHole_2.2mm_M2
- moved D2 15.1 mm to (112.1, 101.1), turned to -90 degrees
- moved D3 15.0 mm to (114.5, 86.3)
- turned C8 to 180 degrees
Connections:
- C1 pad 1: Net-(D1-A1) -> +3.3V
- C2 pad 1: Net-(D1-A1) -> +3.3V
- U1 pad 1: Net-(D1-A1) -> +3.3V
- U1 pad 3: Net-(D1-A1) -> +3.3V
Routing:
- net GND: track 0.00 -> 16.9 mm, vias 0 -> 22
- net +3.3V: track 0.00 -> 10.3 mm
- net Net-(J1-CC2): track 0.00 -> 8.73 mm, vias 0 -> 2
- net Net-(J1-CC1): track 0.00 -> 7.85 mm, vias 0 -> 2
- net Net-(J1-VBUS): track 0.00 -> 4.44 mm
- added copper zone on F.Cu, net +1V8
- added copper zone on F.Cu, net +3.3V
- added copper zone on F.Cu, net +5V
- added copper zone on B.Cu, net GND
- added copper zone on F.Cu, net GND
- added copper zone on F.Cu, net Net-(D1-A1)
- added copper zone on F.Cu, net Net-(D2-A)
- added copper zone on F.Cu, net Net-(D3-A)
- added copper zone on F.Cu, net Net-(D4-A)
- added copper zone on F.Cu, net Net-(J1-VBUS)
Other:
- board size 30 x 18.5 mm -> 30.8 x 18.5 mm
