File: MiniBench/MiniBench.kicad_sch (KiCad schematic)
At the start: 27 parts, among them J1 10174819-00011LF, J3 Screw_Terminal_01x04, U1 AP2112K-1.8, U2 AMS1117-3.3

Commit message: Update README
Parts:
- removed H1, H2: M2, MountingHole:MountingHole_2.2mm_M2, symbol Mechanical:MountingHole
Connections:
- net +3.3V: now also C1.1, C2.1, U1.1 (VIN), U1.3 (EN)
- net at C3.1, C5.1, C6.1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: no longer C1.1, C2.1, U1.1 (VIN), U1.3 (EN)
Other:
- note removed: "IP_min = 15W"
- moved on the sheet: J3
